Commit message: Add head camera publisher and ChArUco camera calibration
openarm_camera publishes the HBV USB head camera: MJPEG frames passed
through on image_raw/compressed, image_raw decoded on demand, camera_info
from an intrinsics NPZ. The Sagres URDF gets camera_optical_frame under
camera_link.

scripts/calibrate_intrinsics.py and scripts/calibrate_handeye.py calibrate
from rosbags of the ChArUco board: intrinsics, and the eye-to-hand camera
pose from /tf with the board on a gripper (closed-form AX = XB plus a
reprojection refinement; OpenCV 5's Python bindings lack calibrateHandEye).

Co-Authored-By: Claude Opus 5.5 <noreply@anthropic.com>

File: src/openarm_ee_control/urdf/sagres_openarm_v10.urdf.xacro (robot description, xacro)
@@ -19,5 +19,6 @@
   * motor gains from openarm_ee_control/config/control_gains_v10.yaml (control_gains_file arg)
   * camera_link, fixed to world at the pose used by ros2ws/.../robot_bringup.launch.py
-    (disable with camera:=false if a separate static TF publishes it)
+    (disable with camera:=false if a separate static TF publishes it), and its child
+    camera_optical_frame; scripts/calibrate_handeye.py prints the calibrated camera_xyz/rpy
 -->
 <robot xmlns:xacro="http://www.ros.org/wiki/xacro" name="openarm">
@@ -104,4 +105,12 @@
       <origin xyz="$(arg camera_xyz)" rpy="$(arg camera_rpy)" />
     </joint>
+    <!-- REP 103: camera_link x forward, z up; the optical frame (z forward, x right, y down)
+         is the frame_id of the openarm_camera images -->
+    <link name="camera_optical_frame" />
+    <joint name="camera_link_to_optical" type="fixed">
+      <parent link="camera_link" />
+      <child link="camera_optical_frame" />
+      <origin xyz="0 0 0" rpy="${-pi/2} 0 ${-pi/2}" />
+    </joint>
   </xacro:if>
 </robot>
